File: 00-proyecto-02/grupo-02/secuenciador-02-v02/4015-falstad.kicad_sch (KiCad schematic)
At the start: 42 parts, among them J1 Barrel_Jack_Switch, J10 AudioJack2_SwitchT, J11 AudioJack2_SwitchT, J12 AudioJack2_SwitchT, J3 Barrel_Jack_Switch, J6 AudioJack2_SwitchT, J7 AudioJack2_SwitchT, J8 AudioJack2_SwitchT, J9 AudioJack2_SwitchT, Q1 PN2222A, Q2 PN2222A, Q3 PN2222A, Q4 PN2222A, Q5 PN2222A, Q6 PN2222A, SW3 SW_SPDT, U1 4040, U3 L7805

Commit message: Add files via upload
Parts:
- removed C4: 100u, Capacitor_THT:CP_Radial_D8.0mm_P3.80mm, symbol Device:C_Polarized
- removed C5: 10u, Capacitor_THT:CP_Radial_D4.0mm_P2.00mm, symbol Device:C_Polarized
- removed C6: 100n, Capacitor_THT:C_Disc_D5.0mm_W2.5mm_P2.50mm, symbol Device:C
- removed D10, D11, D13, D14, D9: LED, LED_THT:LED_D5.0mm, symbol Device:LED
- removed D6: 1N4007, Diode_THT:D_DO-41_SOD81_P10.16mm_Horizontal, symbol Diode:1N4007
- removed J1, J3: Barrel_Jack_Switch, Connector_BarrelJack:BarrelJack_Horizontal, symbol Connector:Barrel_Jack_Switch
- removed Q1, Q2: PN2222A, Package_TO_SOT_THT:TO-92_Inline, symbol Transistor_BJT:PN2222A
- removed R10, R14: 1k, Resistor_THT:R_Axial_DIN0207_L6.3mm_D2.5mm_P10.16mm_Horizontal, symbol Device:R
- removed SW3: SW_SPDT, dis8644:spdt_ssd12d00g3, symbol Switch:SW_SPDT
- removed U1: 4040, Package_DIP:DIP-16_W7.62mm, symbol 4xxx:4040
- removed U3: L7805, Package_TO_SOT_THT:TO-220-3_Horizontal_TabDown, symbol Regulator_Linear:L7805
- added C7: 100u, Capacitor_THT:CP_Radial_D8.0mm_P3.80mm, symbol Device:C_Polarized
- added C8: 10u, Capacitor_THT:CP_Radial_D4.0mm_P2.00mm, symbol Device:C_Polarized
- added C9: 100n, Capacitor_THT:C_Disc_D5.0mm_W2.5mm_P2.50mm, symbol Device:C
- added D1, D2, D3, D4, D5, D6, D7: LED, LED_THT:LED_D5.0mm, symbol Device:LED
- added D11: 1N4007, Diode_THT:D_DO-41_SOD81_P10.16mm_Horizontal, symbol Diode:1N4007
- added J13, J14: AudioJack2_SwitchT, dis8644:PJ301M-12, symbol Connector_Audio:AudioJack2_SwitchT
- added J2, J4: Barrel_Jack_Switch, Connector_BarrelJack:BarrelJack_Horizontal, symbol Connector:Barrel_Jack_Switch
- added Q1: BC548, Package_TO_SOT_THT:TO-92_Inline, symbol Transistor_BJT:BC548
- added Q10, Q7, Q8, Q9: PN2222A, Package_TO_SOT_THT:TO-92_Inline, symbol Transistor_BJT:PN2222A
- added R2: 10k, Resistor_THT:R_Axial_DIN0207_L6.3mm_D2.5mm_P10.16mm_Horizontal, symbol Device:R
- added R20, R21, R22, R3: 1k, Resistor_THT:R_Axial_DIN0207_L6.3mm_D2.5mm_P10.16mm_Horizontal, symbol Device:R
- added R4, R5, R6: 220, Resistor_THT:R_Axial_DIN0207_L6.3mm_D2.5mm_P10.16mm_Horizontal, symbol Device:R
- added SW4: SW_SPDT, dis8644:spdt_ssd12d00g3, symbol Switch:SW_SPDT
- added U2: 4015, Package_DIP:DIP-16_W7.62mm_LongPads, symbol 4xxx_IEEE:4015
- added U4: L7805, Package_TO_SOT_THT:TO-220-3_Horizontal_TabDown, symbol Regulator_Linear:L7805
- R11, R13, R7, R8, R9: value 1k -> 220
Connections:
- net +12V: now also C7.1, D11.1 (K), U4.1 (IN)
- net +5V: now also D12.2 (A), C8.1, C9.1, R3.2, U2.16 (Vdd), U2.16 (Vdd), U4.3 (OUT); no longer D8.2 (A)
- net GND: now also D8.1 (K), R12.1, C7.2, C8.2, C9.2, D1.1 (K), D2.1 (K), D3.1 (K), D4.1 (K), D5.1 (K), D6.1 (K), D7.1 (K), J13.1, J14.1, J2.2, J4.2, Q1.3 (E), U2.14 (MR), U2.6 (MR), U2.8 (Vss), U2.8 (Vss), U4.2 (GND); no longer D12.1 (K), R7.1
- net at J6.3: now also U2.1 (CP), U2.9 (CP)
- net at R18.1: now also Q6.2 (B); no longer J12.3
- net at R16.1: now also Q4.2 (B); no longer J11.3
- net at J10.3: now also R18.2, U2.2 (Q4), U2.7 (D)
- net at J9.3: now also R17.2, U2.11 (Q3); no longer R12.1
- net at J8.3: now also R16.2, U2.12 (Q2)
- net at J7.3: now also R15.2, U2.13 (Q1); no longer R8.1
- net at R7.2: now also Q6.3 (C); no longer D8.1 (K)
- net at Q4.3 (C): now also R5.2; no longer R15.1
- net at R11.1: now also D7.2 (A)
- net at R11.2: now also Q9.3 (C)
- net at R17.1: now also Q5.2 (B); no longer Q5.3 (C)
- net at R19.1: now also Q7.2 (B); no longer Q6.3 (C)
- net at R19.2: now also J11.3, U2.5 (Q1)
- net at R12.2: now also D12.1 (K); no longer Q3.2 (B)
- net at R9.2: now also Q8.3 (C)
- net at R9.1: now also D6.2 (A)
- net at R8.2: now also Q7.3 (C)
- net at R13.1: now also D8.2 (A); no longer Q3.3 (C)
- net at R13.2: now also Q10.3 (C)
- new net: Q1.1 (C), R3.1, U2.15 (D)
- new net: D3.2 (A), R6.1
- new net: D1.2 (A), R4.1
- new net: J2.1, J4.1, SW4.1 (A)
- new net: Q9.2 (B), R21.1
- new net: Q10.2 (B), R22.1
- new net: J12.3, R20.2, U2.4 (Q2)
- new net: D5.2 (A), R8.1
- new net: D2.2 (A), R5.1
- new net: J13.3, R21.2, U2.3 (Q3)
- new net: J14.3, R2.2, R22.2, U2.10 (Q4)
- new net: Q3.3 (C), R4.2
- new net: Q3.2 (B), R15.1
- new net: Q1.2 (B), R2.1
- new net: D4.2 (A), R7.1
- new net: Q8.2 (B), R20.1
- new net: D11.2 (A), SW4.2 (B)
- new net: Q5.3 (C), R6.2
- no-connect marks 16 -> 12
